File: elec/layout/default/jst-gh.kicad_pcb (KiCad board)
At the start: 2 copper layers, 225.7 x 100.8 mm, 0 parts

Commit message: layout
Parts:
- added J1: , lib:CONN-SMD_4P-P1.25_SM04B-GHS-TB-LF-SN, F.Cu at (163.9, 102.5)
Changed lines of the file:
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@@
   )
   (net 0 "")
+  (net 1 "gnd")
+  (net 2 "canl")
+  (net 3 "canh")
+  (net 4 "vcc")
+  (footprint "lib:CONN-SMD_4P-P1.25_SM04B-GHS-TB-LF-SN" (layer "F.Cu")
+    (at 163.92 102.54)
+    (attr smd)
+    (fp_text reference "J1" (at 3.5567 -2.607997) (layer "F.SilkS")
+        (effects (font (size 1 1) (thickness 0.15)))
+    )
+    (fp_text value "" (at 0 5.6) (layer "F.Fab")
+        (effects (font (size 1 1) (thickness 0.15)))
+    )
+    (fp_text user "${REFERENCE}" (at 0 0) (layer "F.Fab")
+        (effects (font (size 1 1) (thickness 0.15)))
+    )
+    (fp_line (start -4.27 -1.69) (end -4.27 -0.04)
+      (stroke (width 0.25) (type solid)) (layer "F.SilkS"))
+    (fp_line (start -3 2.71) (end 2.92 2.71)
+      (stroke (width 0.25) (type solid)) (layer "F.SilkS"))
+    (fp_line (start -2.36 -1.69) (end -4.27 -1.69)
+      (stroke (width 0.25) (type solid)) (layer "F.SilkS"))
+    (fp_line (start 2.34 -1.68) (end 4.28 -1.68)
+      (stroke (width 0.25) (type solid)) (layer "F.SilkS"))
+    (fp_line (start 4.28 -1.68) (end 4.28 0.02)
+      (stroke (width 0.25) (type solid)) (layer "F.SilkS"))
+    (fp_circle (center -3.44 -2.1) (end -3.32 -2.1)
+      (stroke (width 0.25) (type solid)) (fill none) (layer "F.SilkS"))
+    (fp_circle (center -1.89 -1.13) (end -1.77 -1.13)
+      (stroke (width 0.25) (type solid)) (fill none) (layer "Cmts.User"))
+    (fp_circle (center -4.12 -2.28) (end -4.09 -2.28)
+      (stroke (width 0.06) (type solid)) (fill none) (layer "F.Fab"))
+    (pad "1" smd rect (at -1.88 -1.6) (size 0.6 1.7) (layers "F.Cu" "F.Paste" "F.Mask")
+      (net 4 "vcc") (pintype "stereo"))
+    (pad "2" smd rect (at -0.63 -1.6) (size 0.6 1.7) (layers "F.Cu" "F.Paste" "F.Mask")
+      (net 3 "canh") (pintype "stereo"))
+    (pad "3" smd rect (at 0.62 -1.6) (size 0.6 1.7) (layers "F.Cu" "F.Paste" "F.Mask")
+      (net 2 "canl") (pintype "stereo"))
+    (pad "4" smd rect (at 1.87 -1.6) (size 0.6 1.7) (layers "F.Cu" "F.Paste" "F.Mask")
+      (net 1 "gnd") (pintype "stereo"))
+    (pad "5" smd rect (at 3.72 1.6) (size 1 2.7) (layers "F.Cu" "F.Paste" "F.Mask"))
+    (pad "6" smd rect (at -3.72 1.6) (size 1 2.7) (layers "F.Cu" "F.Paste" "F.Mask"))
+    (model "/Users/narayanpowderly/Documents/atopile-workspace/servo-drive/.ato/modules/jst-gh/elec/footprints/footprints.3dshapes/CONN-SMD_GH1.25-WS-4P.wrl"
+      (offset (xyz 0 -0.15 -0))
+      (scale (xyz 1 1 1))
+      (rotate (xyz 0 0 0))
+    )
+  )
   (gr_circle (center 225.62 81.79) (end 227.32 81.79)
     (stroke (width 0.1) (type solid)) (fill none) (layer "Edge.Cuts"))
@@
       (xy 69.100734 49.778315)
     )
-    (stroke (width 0) (type solid)) (fill none) (layer "Edge.Cuts"))
+    (stroke (width 0.1) (type solid)) (fill none) (layer "Edge.Cuts"))
   (gr_arc (start 261.62 113.79) (mid 260.448427 116.618427) (end 257.62 117.79)
     (stroke (width 0.1) (type solid)) (layer "Edge.Cuts"))
